File: LVPWR.kicad_sch (KiCad schematic)
At the start: 21 parts, among them U4 LMR51610XDBVR, U5 LMR51610XDBVR, U9 ADPL44002AUJZ-1.8-R7

Commit message: Add Doc
Parts:
- removed C40, C41: GRM21BR71E225KE11L, CAP_GRM21BR61H106KE43K_MUR, symbol 2025-04-06_15-56-13:GRM21BR61H106KE43K
- removed U9: ADPL44002AUJZ-1.8-R7, UJ-5_ADI, symbol 2025-06-28_14-44-19:ADPL44002AUJZ-1.8-R7
